File: hdw/TQFP48/TQFP48.kicad_pcb (KiCad board)
At the start: 2 copper layers, 61 x 17.8 mm, 3 parts, among them J1 Conn_01x24, J2 Conn_01x24, U1 TQFP48

Commit message: Save changes at: 1748380927
Routing:
- net P36: track 2.84 -> 3.36 mm
- net P13: track 2.84 -> 3.36 mm
- net P37: track 2.84 -> 3.36 mm
- net P12: track 2.84 -> 3.36 mm
- removed copper zone on B.Cu, net (none)
- removed copper zone on F.Cu, net (none)
Other:
- board text added: "31"
- board text added: "32"
- board text added: "33"
- board text added: "34"
- board text added: "35"
- board text added: "38"
- board text added: "39"
- board text added: "40"
- board text added: "41"
- board text added: "42"
- board text added: "43"
- board text added: "44"
- board text added: "45"
- board text added: "46"
- board text added: "47"

Commit message: Save changes at: 1748616972
Other:
- board text added: "17"
- board text removed: "13"
Changed lines of the file:
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@@
 	)
 	(gr_text "15"
+		(at 99.06 63.754 0)
+		(layer "F.SilkS")
+		(effects
+			(font
+				(size 1 1)
+				(thickness 0.15)
+			)
+		)
+	)
+	(gr_text "16"
 		(at 101.6 63.754 0)
-		(layer "F.SilkS")
-		(effects
-			(font
-				(size 1 1)
-				(thickness 0.15)
-			)
-		)
-	)
-	(gr_text "16"
-		(at 104.14 63.754 0)
 		(layer "F.SilkS")
 		(effects
@@
 	)
 	(gr_text "14"
-		(at 99.06 63.754 0)
+		(at 96.52 63.754 0)
 		(layer "F.SilkS")
 		(effects
@@
 		)
 	)
-	(gr_text "13"
-		(at 96.52 63.754 0)
-		(layer "F.SilkS")
-		(effects
+	(gr_text "17"
+		(at 104.14 63.754 0)
+		(layer "F.SilkS")
+		(effects
