File: hdw/USBC2/USBC2.kicad_pcb (KiCad board)
At the start: 2 copper layers, 14 x 17.8 mm, 7 parts, among them J1 Conn_01x02, J2 Conn_01x02, J3 Conn_01x02, J4 Conn_01x02, P1 USB_C_Receptacle_USB2.0

Commit message: Save changes at: 1748195240
Parts:
- added J5: Conn_01x02, Connector_PinHeader_2.54mm:PinHeader_1x02_P2.54mm_Vertical, B.Cu at (88.9, 129.5)
- added J6: Conn_01x02, Connector_PinHeader_2.54mm:PinHeader_1x02_P2.54mm_Vertical, B.Cu at (88.9, 109.2)
- J1, J2, J3, J4, R1, R2: moved to B.Cu
- P1: value USB_C_Receptacle_USB2.0 -> USB_C_2.0; footprint Connector_USB:USB_C_Receptacle_GCT_USB4105-xx-A_16P_TopMnt_Horizontal -> Connector_USB:USB_C_Receptacle_GCT_USB4085
- moved R2 9.65 mm to (85.7, 119.1), turned to 90 degrees
- moved P1 3.65 mm to (89.8, 116.4)
- moved R1 2.98 mm to (92.7, 119.7), turned to -90 degrees
- moved J4 2.54 mm to (96.5, 127.0)
- moved J3 2.54 mm to (96.5, 111.8)
- turned J1 to -90 degrees
- turned J2 to -90 degrees
Routing:
- net GND: track 16.6 -> 0.00 mm
- net D-: track 28.2 -> 21.3 mm
- net D+: track 36.7 -> 32.0 mm
- net Net-(P1-CC1): track 2.40 -> 2.96 mm
Other:
- board size 14 x 17.8 mm -> 14 x 22.9 mm
